File: Power.kicad_sch (KiCad schematic)
At the start: 33 parts, among them U2 AXP223_C2997893

Commit message: changed some ethernet stuff
Parts:
- gave numbers to parts that had none: 1

Commit message: power changes
Parts:
- removed C14: 4.7uF, symbol Device:C
- added C41, C43, C44, C45, C46, C47, C48, C49, C50, C53: 10uF, symbol Device:C
- added C42: 0.1uF, symbol Device:C
- added C51, C52: 1uF, symbol Device:C
- added L6: 1.5uH, symbol Device:L
- added Q1: WPM1481-6/TR, easyeda2kicad:DFN-6L_L2.0-W2.0-P0.65-BL_WPM1481-6, symbol easyeda2kicad:WPM1481-6_TR
- added R10, R8, R9: 10mR, symbol Device:R
- added R11, R12: 2.2K, symbol Device:R
- added R13: 51K, symbol Device:R
Connections:
- net GND: now also U2.59 (PGND_CHG), C41.1, C42.1, C43.1, C44.1, C45.1, C46.1, C47.1, C48.1, C49.1, C50.2, C53.2, R9.1
- net IPSOUT: now reaches C3.2, U2.39 (VIN3)
- net IPSOUT: now also C1.2, C2.2, U2.1 (ELDOIN), U2.13 (VIN1), U2.18 (DLDOIN), U2.23 (VIN2), U2.33 (ALDOIN), U2.53 (PS), U2.54 (PS), U2.62 (VIN_CHG), U2.63 (VIN_CHG), C43.2, C44.2, C45.2, C48.2, Q1.4 (S), Q1.7 (S)
- net VCC_RTC: now reaches U2.46 (VCC_RTC)
- net VCC_RTC: now also U2.11 (N_VBUSEN), R11.2, R12.2, R13.2
- net VCC_3V3_ANALOG: now reaches U1.V3 (AVCC)
- net VCC_3V3_ANALOG: now also U2.32 (ALDO1), C41.2, C42.2
- net PWR_ON: now reaches U2.12 (PWRON)
- net ELDO2: now reaches U2.2 (ELDO2)
- net AXP_IRQ: now reaches U2.29 (IRQ)
- net AXP_IRQ: now also R13.1
- net ELDO3: now reaches U2.3 (ELDO3)
- net NTC: now reaches U2.30 (TS)
- net NTC: now also R9.2
- net at U2.31 (GPIO1/PWREN): now also C47.2
- net at U2.37 (GPIO0): now also C46.2
- net AXP_PWROK: now reaches U2.43 (PWROK)
- net AXP_SCL: now reaches U2.44 (SCK)
- net AXP_SCL: now also R11.1
- net AXP_SDA: now reaches U2.45 (SDA)
- net AXP_SDA: now also R12.1
- net +BATT: now reaches U2.49 (BATSENCE)
- net +BATT: now also C52.2, C53.1, R10.2
- net CHSENCEN: now reaches U2.50 (LOADSENCE)
- net CHSENCEN: now also U2.58 (CHSENCEN), C50.1, C51.2, C52.1, Q1.1 (D), Q1.2 (D), Q1.5 (D), Q1.6 (D), Q1.8 (D), R10.1, R8.2
- net N_BATDRV: now reaches U2.51 (N_BATDRV)
- net N_BATDRV: now also Q1.3 (G)
- net CHG_LED: now reaches U2.52 (CHGLED)
- net CHSENCEP: now reaches U2.57 (CHSENCEP)
- net CHSENCEP: now also C49.2, C51.1, L6.1, R8.1
- net LX_CHG: now reaches U2.60 (LX_CHG)
- net LX_CHG: now also U2.61 (LX_CHG), L6.2
- net ELDO1: now reaches U2.68 (ELDO1)
- no-connect marks 5 -> 7
Other:
- moved on the sheet: C1, C10, C11, C12, C13, C2, C27, C28, C29, C3, C30, C31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

Commit message: power changes and pinout update
Parts:
- added C54, C55, C56, C57, C58, C59, C60: 0.1uF, symbol Device:C
Connections:
- net GND: now also U1.M5 (HGND), U1.U3 (AGND), C54.1, C55.1, C56.1, C57.1, C58.1, C59.1, C60.1
- net VCC3V3: now also U1.G10 (VDD_EFUSE), U1.G7 (EPHY_VCC), U1.H7 (VCC_PG), U1.J15 (VCC_PD), U1.J6 (HVCC), U1.N3 (VCC_PLL), C56.2, C57.2, C58.2, C59.2, C60.2
- net VCC_RTC: now also U1.K6 (VCC_RTC)
- net at U1.H11 (VDD_EF_USEBP): now also C54.2
Other:
- moved on the sheet: C35, C36, U1D, U1E, U1F

Commit message: power things, minor changes
Parts:
- added C14, C64: 10uF, symbol Device:C
- added C61: 4.7uF, symbol Device:C
- added C62: 0.1uF, symbol Device:C
- added C63: 1uF, symbol Device:C
- added C65: 1nF, symbol Device:C
- added L7: 1.5uH, symbol Device:L
- C58: value 0.1uF -> 1uF
Connections:
- net VCC_3V3_ANALOG is gone; now on net VCC3V3_AUDIO: C41.2, C42.2, U1.V3 (AVCC), U2.32 (ALDO1)
- net GND: now also U1.T9 (GND-CPUFB), U2.66 (PGND4), C14.1, C61.1, C62.1, C63.1, C64.1, C65.1
- net IPSOUT: now also U2.64 (VIN4), C14.2
- net VCC1V2_CPU: now also U1.M4 (RTC_VIO), C61.2; no longer U2.28 (DCDC2)
- net VCC1V2_SYS: now also C55.2, U1.F8 (EPHY_VDD)
- net CPUX_FB: now reaches U1.T10 (GND-CPUFB)
- net CPUX_FB: now also U2.28 (DCDC2)
- net at U2.65 (LX4): now also L7.1
- net DCDC4: now reaches U2.67 (DCDC4)
- net DCDC4: now also C64.2, C65.2, L7.2
- net VCC3V3_AUDIO: now reaches U1.G9 (V33_TV)
- net VCC3V3_AUDIO: now also C62.2, C63.2
- no-connect marks 7 -> 3
Other:
- moved on the sheet: C27, C28, C29, C30, C35, C36, C55, C56, C57, C58, C59, C60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

Commit message: minor changes
Parts:
- added C70, C71: 22uF, symbol Device:C
- added C72, C73, C76, C81: 10uF, symbol Device:C
- added C74, C77, C78, C82, C83: 1uF, symbol Device:C
- added C75, C79, C80, C84, C85, C86: 0.1uF, symbol Device:C
Connections:
- net +5V: now also C70.1, C71.1, C72.1
- net GND: now also C70.2, C71.2, C72.2, C73.2, C74.2, C75.2, C76.2, C77.2, C78.2, C79.2, C80.2, C81.2, C82.2, C83.2, C84.2, C85.2, C86.2
- net VCC1V2_CPU: now also C76.1, C77.1, C78.1, C79.1, C80.1
- net VCC1V2_SYS: now also C81.1, C82.1, C83.1, C84.1, C85.1
- net VCC3V3: now also C73.1, C74.1, C75.1
- net VCC_RTC: now also C86.1
Other:
- moved on the sheet: C1, C10, C13, C2, C3, C4, C5, C6, C7, C8, C9, L1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
