File: Ethernet.kicad_sch (KiCad schematic)
At the start: 2 parts, among them J1 HR911105A_C12074, U1 H3

Commit message: changed some ethernet stuff
Parts:
- removed J1: HR911105A_C12074, easyeda2kicad:RJ45-TH_HR911105A, symbol easyeda2kicad:HR911105A_C12074
- added C37, C39: 0.1uF, symbol Device:C
- added C38, C40: 4.7uF, symbol Device:C
- added L5: 2.2uH, symbol Device:L
- added R7: 2K49, symbol Device:R
- added RJ1: R-RJ45R08P-C000, easyeda2kicad:RJ45-TH_R-RJ45R08P-C000, symbol easyeda2kicad:R-RJ45R08P-C000
- added U9: RTL8211E-VB-CG, easyeda2kicad:QFN-48_L6.0-W6.0-P0.40-BL-EP3.8, symbol easyeda2kicad:RTL8211E-VB-CG
Connections:
- net RGMII_MDC: now also U9.30 (MDC)
- net RGMII_RXCK: now also U9.19 (RXC)
- net RGMII_RXCTL: now also U9.13 (RXCTL/PHY_AD)
- net RGMII_RXD0: now also U9.14 (RXD[0]/SELRGV)
- net RGMII_RXD1: now also U9.16 (RXD[1]/TXDLY)
- net RGMII_RXD2: now also U9.17 (RXD[2]/AN0)
- net RGMII_RXD3: now also U9.18 (RXD[3]/AN1)
- net RGMII_TXCK: now also U9.22 (TXC)
- net RGMII_TXCTL: now also U9.27 (TXCTL)
- net RGMII_TXD0: now also U9.23 (TXD[0])
- net RGMII_TXD1: now also U9.24 (TXD[1])
- net RGMII_TXD2: now also U9.25 (TXD[2])
- net RGMII_TXD3: now also U9.26 (TXD[3])
- net MDIO renamed RGMII_MDIO
- net RGMII_MDIO: now also U9.31 (MDIO)
- new net: R7.2, U9.39 (RSET)
- new net: L5.2, U9.48 (REG_OUT)
- new net AVDD10: C39.2, C40.2, L5.1, U9.28 (DVDD10), U9.3 (AVDD10), U9.36 (DVDD10), U9.40 (AVDD10), U9.9 (AVDD10)
- new net ENET_LED0: U9.34 (LED0/PHY_AD0)
- new net ENET_LED1: U9.35 (LED1/PHY_AD1)
- new net ENET_LED2: U9.32 (LED2/RXDLY)
- new net ENET_MDI0+: U9.1 (MDI[0]+)
- new net ENET_MDI0-: U9.2 (MDI[0]-)
- new net ENET_MDI1+: U9.4 (MDI[1]+)
- new net ENET_MDI1-: U9.5 (MDI[1]-)
- new net ENET_MDI2+: U9.7 (MDI[2]+)
- new net ENET_MDI2-: U9.8 (MDI[2]-)
- new net ENET_MDI3+: U9.10 (MDI[3]+)
- new net ENET_MDI3-: U9.11 (MDI[3]-)
- new net GND: C37.2, C38.2, C39.1, C40.1, R7.1, U9.47 (GND), U9.49 (EPAD)
- new net VCC3V3_ENET: C37.1, C38.1, U9.44 (VDDREG), U9.45 (VDDREG)
- no-connect marks 3 -> 4

Commit message: minor changes
Parts:
- removed RJ1: R-RJ45R08P-C000, easyeda2kicad:RJ45-TH_R-RJ45R08P-C000, symbol easyeda2kicad:R-RJ45R08P-C000
Changed lines of the file:
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@@
 		(fields_autoplaced yes)
 		(property "Reference" "U1"
-			(at 76.2 43.18 0)
+			(at 53.34 45.72 0)
 			(effects
 				(font
@@
 		)
 		(property "Value" "H3"
-			(at 76.2 45.72 0)
+			(at 53.34 48.26 0)
 			(effects
 				(font
@@
 		)
 		(instances
-			(project "H3_SBC"
+			(project ""
+				(path "/2511caf5-b791-49bc-bcf7-734707cf883b"
+					(reference "U1")
+					(unit 9)
+				)
 				(path "/2511caf5-b791-49bc-bcf7-734707cf883b/35bec0f3-f97e-4602-a3cd-7982e33e73da"
 					(reference "U1")
@@
 					(unit 1)
 				)
-			)
-		)
-	)
-	(symbol
-		(lib_id "easyeda2kicad:R-RJ45R08P-C000")
-		(at 81.28 142.24 0)
-		(unit 1)
-		(exclude_from_sim no)
-		(in_bom yes)
-		(on_board yes)
-		(dnp no)
-		(fields_autoplaced yes)
-		(property "Reference" "RJ1"
-			(at 101.6 133.2798 0)
-			(effects
-				(font
-					(size 1.27 1.27)
-				)
-			)
-		)
-		(property "Value" "R-RJ45R08P-C000"
-			(at 101.6 135.8198 0)
-			(effects
-				(font
-					(size 1.27 1.27)
-				)
-			)
-		)
-		(property "Footprint" "easyeda2kicad:RJ45-TH_R-RJ45R08P-C000"
-			(at 81.28 162.56 0)
-			(effects
-				(font
-					(size 1.27 1.27)
-				)
-				(hide yes)
-			)
-		)
-		(property "Datasheet" "https://lcsc.com/product-detail/Ethernet-Connectors-Modular-Connectors-RJ45-RJ11_Shenzhen-Cankemeng-R-RJ45R08P-C000_C386757.html"
-			(at 81.28 165.1 0)
-			(effects
-				(font
-					(size 1.27 1.27)
-				)
-				(hide yes)
-			)
-		)
-		(property "Description" ""
-			(at 81.28 142.24 0)
-			(effects
-				(font
-					(size 1.27 1.27)
-				)
-				(hide yes)
-			)
-		)
-		(property "LCSC Part" "C386757"
-			(at 81.28 167.64 0)
-			(effects
-				(font
-					(size 1.27 1.27)
-				)
-				(hide yes)
-			)
-		)
-		(pin "6"
-		)
-		(pin "10"
-		)
-		(pin "7"
-		)
-		(pin "13"
-		)
-		(pin "8"
-		)
-		(pin "9"
-		)
-		(pin "12"
-		)
-		(pin "11"
-		)
-		(pin "2"
-		)
-		(pin "3"
-		)
-		(pin "4"
-		)
-		(pin "1"
-		)
-		(pin "5"
-		)
-		(pin "14"
-		)
-		(instances
-			(project ""
-				(path "/2511caf5-b791-49bc-bcf7-734707cf883b/35bec0f3-f97e-4602-a3cd-7982e33e73da"
-					(reference "RJ1")
-					(unit 1)
-				)

Commit message: recovered ethernet power changes
Parts:
- added C123, C125: 27pF, symbol Device:C
- added C124, C126, C127, C130: 0.1uF, symbol Device:C
- added C128, C129: 4.7uF, symbol Device:C
- added R23: 20K, symbol Device:R
- added R24, R25, R26: 4K7, symbol Device:R
- added R27: 0R, symbol Device:R
- added U5: AP2127K-2.5, Package_TO_SOT_SMD:SOT-23-5, symbol Regulator_Linear:AP2127K-2.5
- added X3: 5YAA25000121TF25E2, easyeda2kicad:CRYSTAL-SMD_4P-L3.2-W2.5-BL, symbol easyeda2kicad:5YAA25000121TF25E2
Connections:
- net GND: now also C123.1, C124.1, C125.1, C126.1, C127.1, C128.1, C129.1, C130.1, R23.2, U5.2 (GND), X3.2 (GND), X3.4 (GND)
- net RGMII_CLKIN: now also R27.1
- net VCC3V3_ENET: now also U9.37 (DVDD33), U9.38 (ENSWREG), U9.41 (AVDD33), U9.6 (AVDD33), C127.2, C128.2, C129.2, R24.2, R25.2, R26.1
- net at U9.20 (INTB): now also R25.1
- net DVDD25: now reaches U9.21 (DVDD33)
- net DVDD25: now also C126.2, U5.5 (VOUT)
- net PHYRSTB: now reaches U9.29 (PHYRSTB)
- net PHYRSTB: now also C130.2, R24.1
- net at U9.33 (PMEB): now also R26.2
- net CKXTAL_OUT: now reaches U9.42 (CKXTAL1)
- net CKXTAL_OUT: now also C125.2, X3.3
- net CKXTAL_IN: now reaches U9.43 (CKXTAL2)
- net CKXTAL_IN: now also C123.2, X3.1
- net at U9.46 (CLK125): now also R27.2
- new net +5V: C124.2, U5.1 (VIN)
- new net EMAC_PWR_EN: R23.1, U5.3 (EN)
Other:
- moved on the sheet: U1I

Commit message: linking symbols to footprints
Parts:
- C123, C125: footprint (none) -> Capacitor_SMD:C_0402_1005Metric
- C124, C126, C127, C128, C129, C130, C37, C38, C39, C40: footprint (none) -> Capacitor_SMD:C_0603_1608Metric
- L5: footprint (none) -> Inductor_SMD:L_0402_1005Metric
- R23, R24, R25, R26, R27, R7: footprint (none) -> Resistor_SMD:R_0402_1005Metric
- U1: footprint BGA347_H3_AWT -> (none)
Changed lines of the file:
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@@
 			)
 		)
-		(property "Footprint" ""
+		(property "Footprint" "Resistor_SMD:R_0402_1005Metric"
 			(at 219.71 137.922 90)
 			(effects
@@
 			)
 		)
-		(property "Footprint" "BGA347_H3_AWT"
+		(property "Footprint" ""
 			(at -3.81 29.21 0)
 			(effects
@@
 			)
 		)
-		(property "Footprint" ""
+		(property "Footprint" "Capacitor_SMD:C_0603_1608Metric"
 			(at 165.4048 46.99 0)
 			(effects
@@
 			)
 		)
-		(property "Footprint" ""
+		(property "Footprint" "Resistor_SMD:R_0402_1005Metric"
 			(at 179.07 31.242 90)
 			(effects
@@
 			)
 		)
-		(property "Footprint" ""
+		(property "Footprint" "Capacitor_SMD:C_0603_1608Metric"
 			(at 210.82 24.4348 0)
 			(effects
@@
 			)
 		)
-		(property "Footprint" ""
+		(property "Footprint" "Resistor_SMD:R_0402_1005Metric"
 			(at 46.482 179.07 90)
 			(effects
@@
 			)
 		)
-		(property "Footprint" ""
+		(property "Footprint" "Capacitor_SMD:C_0603_1608Metric"
 			(at 124.7648 59.69 0)
 			(effects
@@
 			)
 		)
-		(property "Footprint" ""
+		(property "Footprint" "Capacitor_SMD:C_0603_1608Metric"
 			(at 172.4152 46.99 0)
 			(effects
@@
 			)
 		)
-		(property "Footprint" ""
+		(property "Footprint" "Capacitor_SMD:C_0603_1608Metric"
 			(at 129.8448 146.05 0)
 			(effects
@@
 			)
 		)
-		(property "Footprint" ""
+		(property "Footprint" "Resistor_SMD:R_0402_1005Metric"
 			(at 264.922 69.85 90)
 			(effects
@@
 			)
 		)
-		(property "Footprint" ""
+		(property "Footprint" "Capacitor_SMD:C_0603_1608Metric"
 			(at 86.6648 175.26 0)
 			(effects
@@
 			)
 		)
-		(property "Footprint" ""
+		(property "Footprint" "Resistor_SMD:R_0402_1005Metric"
 			(at 215.392 36.83 90)
 			(effects
@@
 			)
 		)
-		(property "Footprint" ""
+		(property "Footprint" "Capacitor_SMD:C_0402_1005Metric"
 			(at 82.2452 123.19 0)
 			(effects
@@
 			)
 		)
-		(property "Footprint" ""
+		(property "Footprint" "Inductor_SMD:L_0402_1005Metric"
 			(at 186.69 41.91 0)
 			(effects
@@
 			)
 		)
-		(property "Footprint" ""
+		(property "Footprint" "Capacitor_SMD:C_0402_1005Metric"
 			(at 49.8348 123.19 0)
 			(effects
@@
 			)
 		)
-		(property "Footprint" ""
+		(property "Footprint" "Capacitor_SMD:C_0603_1608Metric"
 			(at 57.4548 175.26 0)
 			(effects
@@
 			)
 		)
-		(property "Footprint" ""
+		(property "Footprint" "Capacitor_SMD:C_0603_1608Metric"
 			(at 136.8552 146.05 0)
 			(effects
@@
 			)
 		)
-		(property "Footprint" ""
+		(property "Footprint" "Capacitor_SMD:C_0603_1608Metric"
 			(at 210.82 31.4452 0)
 			(effects
@@
 			)
 		)
-		(property "Footprint" ""
+		(property "Footprint" "Capacitor_SMD:C_0603_1608Metric"
 			(at 147.0152 146.05 0)
 			(effects
@@
 			)
 		)
-		(property "Footprint" ""
+		(property "Footprint" "Resistor_SMD:R_0402_1005Metric"
 			(at 111.252 49.53 90)
 			(effects

Commit message: placed major components
Parts:
- C124, C126, C127, C128, C129, C130, C37, C38, C39, C40: footprint Capacitor_SMD:C_0603_1608Metric -> Capacitor_SMD:C_0402_1005Metric
Changed lines of the file:
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@@
 			)
 		)
-		(property "Footprint" "Capacitor_SMD:C_0603_1608Metric"
+		(property "Footprint" "Capacitor_SMD:C_0402_1005Metric"
 			(at 165.4048 46.99 0)
 			(effects
@@
 			)
 		)
-		(property "Footprint" "Capacitor_SMD:C_0603_1608Metric"
+		(property "Footprint" "Capacitor_SMD:C_0402_1005Metric"
 			(at 210.82 24.4348 0)
 			(effects
@@
 			)
 		)
-		(property "Footprint" "Capacitor_SMD:C_0603_1608Metric"
+		(property "Footprint" "Capacitor_SMD:C_0402_1005Metric"
 			(at 124.7648 59.69 0)
 			(effects
@@
 			)
 		)
-		(property "Footprint" "Capacitor_SMD:C_0603_1608Metric"
+		(property "Footprint" "Capacitor_SMD:C_0402_1005Metric"
 			(at 172.4152 46.99 0)
 			(effects
@@
 			)
 		)
-		(property "Footprint" "Capacitor_SMD:C_0603_1608Metric"
+		(property "Footprint" "Capacitor_SMD:C_0402_1005Metric"
 			(at 129.8448 146.05 0)
 			(effects
@@
 			)
 		)
-		(property "Footprint" "Capacitor_SMD:C_0603_1608Metric"
+		(property "Footprint" "Capacitor_SMD:C_0402_1005Metric"
 			(at 86.6648 175.26 0)
 			(effects
@@
 			)
 		)
-		(property "Footprint" "Capacitor_SMD:C_0603_1608Metric"
+		(property "Footprint" "Capacitor_SMD:C_0402_1005Metric"
 			(at 57.4548 175.26 0)
 			(effects
@@
 			)
 		)
-		(property "Footprint" "Capacitor_SMD:C_0603_1608Metric"
+		(property "Footprint" "Capacitor_SMD:C_0402_1005Metric"
 			(at 136.8552 146.05 0)
 			(effects
@@
 			)
 		)
-		(property "Footprint" "Capacitor_SMD:C_0603_1608Metric"
+		(property "Footprint" "Capacitor_SMD:C_0402_1005Metric"
 			(at 210.82 31.4452 0)
 			(effects
@@
 			)
 		)
-		(property "Footprint" "Capacitor_SMD:C_0603_1608Metric"
+		(property "Footprint" "Capacitor_SMD:C_0402_1005Metric"
 			(at 147.0152 146.05 0)
 			(effects

Commit message: started RAM routing, might move to 1 module though
Parts:
- U1: footprint (none) -> easyeda2kicad:BGA-347_L14.0-W14.0-R21-C21-P0.65-TL
Changed lines of the file:
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@@
 			)
 		)
-		(property "Footprint" ""
+		(property "Footprint" "easyeda2kicad:BGA-347_L14.0-W14.0-R21-C21-P0.65-TL"
 			(at -3.81 29.21 0)
 			(effects

Commit message: routed ethernet and emmc data lines
Connections:
- net DVDD25: now also U9.15 (DVDD33)
Changed lines of the file:
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@@
+	(wire
+		(pts
+			(xy 199.39 114.3) (xy 199.39 115.57)
+		)
+		(stroke
+			(width 0)
+			(type default)
+		)
+	)
 	(wire
 		(pts
@@
 		(effects
 			(font
+				(size 1.27 1.27)
+			)
+			(justify right bottom)
+		)
+	)
+	(label "DVDD25"
+		(at 199.39 115.57 270)
+		(effects
+			(font
