File: H3_SBC-backups/H3_SBC-2025-04-01_232212/H3_SBC.kicad_pcb (KiCad board)
At the start: 6 copper layers, 50 x 40 mm, 14 parts, among them CN1 YXT-BB10-50P-02, CN2 YXT-BB10-50P-02, CN3 YXT-BB10-50P-02, Q1 WPM1481-6/TR, U1 H3, U10 XT28EG32GA4YJECGA, U2 AXP223_C2997893, U3 K4B4G1646E-BYMA 4GB, U4 K4B4G1646E-BYMA 4GB, U5 AP2127K-2.5, U9 RTL8211E-VB-CG, X1 X201232768KLD2SI, X2 SMD-5032_4P 24M 20pf, X3 5YAA25000121TF25E2

Commit message: small fixes
Parts:
- removed Q1: WPM1481-6/TR, easyeda2kicad:DFN-6L_L2.0-W2.0-P0.65-BL_WPM1481-6
- removed U5: AP2127K-2.5, Package_TO_SOT_SMD:SOT-23-5
- removed X2: SMD-5032_4P 24M 20pf, easyeda2kicad:CRYSTAL-SMD_4P-L5.0-W3.2-BL
- removed X3: 5YAA25000121TF25E2, easyeda2kicad:CRYSTAL-SMD_4P-L3.2-W2.5-BL
- added RJ1: R-RJ45R08P-C000, easyeda2kicad:RJ45-TH_R-RJ45R08P-C000, F.Cu at (212.5, 79.1)
- added U8: XOS32024000LT00351005, easyeda2kicad:OSC-SMD_4P-L3.2-W2.5-BL, F.Cu at (187.8, 68.6)
- moved U10 3.28 mm to (176.2, 72.3)
- moved U1 1.58 mm to (176.0, 86.9)
- moved CN2 0.64 mm to (176.1, 95.0)
- turned CN1 to 180 degrees
Connections:
- CN1 pad 18: PG0 -> unconnected-(CN1-Pad18)
- CN1 pad 19: PG1 -> unconnected-(CN1-Pad19)
- CN1 pad 20: PG2 -> unconnected-(CN1-Pad20)
- CN1 pad 21: PG3 -> unconnected-(CN1-Pad21)
- CN1 pad 22: PG4 -> unconnected-(CN1-Pad22)
- CN1 pad 23: PG5 -> unconnected-(CN1-Pad23)
- CN1 pad 24: PG6 -> unconnected-(CN1-Pad24)
- CN1 pad 25: PG7 -> unconnected-(CN1-Pad25)
- CN1 pad 26: CHG_LED -> unconnected-(CN1-Pad26)
- CN1 pad 27: PWR_ON -> unconnected-(CN1-Pad27)
- CN1 pad 28: GND -> unconnected-(CN1-Pad28)
- CN2 pad 17: UBOOT -> unconnected-(CN2-Pad17)
- CN2 pad 18: GND -> unconnected-(CN2-Pad18)
- CN2 pad 19: PG8 -> unconnected-(CN2-Pad19)
- CN2 pad 20: PG9 -> unconnected-(CN2-Pad20)
- CN2 pad 21: GND -> unconnected-(CN2-Pad21)
- CN2 pad 22: DCDC4 -> unconnected-(CN2-Pad22)
- CN2 pad 23: DCDC4 -> unconnected-(CN2-Pad23)
- CN2 pad 24: DCDC4 -> unconnected-(CN2-Pad24)
- CN2 pad 25: DCDC4 -> unconnected-(CN2-Pad25)
- CN2 pad 37: GND -> unconnected-(CN2-Pad37)
- CN2 pad 38: PG11 -> unconnected-(CN2-Pad38)
- CN2 pad 39: PG10 -> unconnected-(CN2-Pad39)
- CN2 pad 40: GND -> unconnected-(CN2-Pad40)
- CN2 pad 41: SPI0_CS -> unconnected-(CN2-Pad41)
- CN2 pad 42: SPI0_CLK -> unconnected-(CN2-Pad42)
- CN2 pad 43: SPI0_MISO -> unconnected-(CN2-Pad43)
- CN2 pad 44: SPI0_MOSI -> unconnected-(CN2-Pad44)
- CN2 pad 45: GND -> unconnected-(CN2-Pad45)
- CN2 pad 46: PA21 -> unconnected-(CN2-Pad46)
- CN2 pad 47: PA20 -> unconnected-(CN2-Pad47)
- CN2 pad 48: PA19 -> unconnected-(CN2-Pad48)
- CN2 pad 49: PA18 -> unconnected-(CN2-Pad49)
- CN2 pad 50: PA17 -> unconnected-(CN2-Pad50)
- CN3 pad 22: GND -> unconnected-(CN3-Pad22)
- CN3 pad 23: TVOUT -> unconnected-(CN3-Pad23)
- CN3 pad 24: GND -> unconnected-(CN3-Pad24)
- CN3 pad 25: PG11 -> unconnected-(CN3-Pad25)
- CN3 pad 26: AXP_PWROK -> unconnected-(CN3-Pad26)
- CN3 pad 27: PWR_ON -> unconnected-(CN3-Pad27)
- CN3 pad 28: ELDO3 -> unconnected-(CN3-Pad28)
- CN3 pad 29: ELDO3 -> unconnected-(CN3-Pad29)
- CN3 pad 30: ELDO2 -> unconnected-(CN3-Pad30)
- CN3 pad 31: ELDO2 -> unconnected-(CN3-Pad31)
- CN3 pad 32: ELDO1 -> unconnected-(CN3-Pad32)
- CN3 pad 33: ELDO1 -> unconnected-(CN3-Pad33)
- CN3 pad 34: NTC -> unconnected-(CN3-Pad34)
- CN3 pad 35: DLDO4 -> unconnected-(CN3-Pad35)
- CN3 pad 36: DLDO4 -> unconnected-(CN3-Pad36)
- CN3 pad 37: DLDO3 -> unconnected-(CN3-Pad37)
- CN3 pad 38: DLDO3 -> unconnected-(CN3-Pad38)
- CN3 pad 39: DLDO2 -> unconnected-(CN3-Pad39)
- CN3 pad 40: DLDO2 -> unconnected-(CN3-Pad40)
- CN3 pad 41: DLDO1 -> SPI0_CS
- CN3 pad 42: DLDO1 -> SPI0_CLK
- CN3 pad 43: +BATT -> SPI0_MISO
- CN3 pad 44: +BATT -> SPI0_MOSI
- CN3 pad 45: +BATT -> GND
- CN3 pad 46: +BATT -> PA21
- CN3 pad 47: +5V -> PA20
- CN3 pad 48: +5V -> PA19
- CN3 pad 49: +5V -> PA18
- CN3 pad 50: +5V -> PA17
- U2 pad 1: /Power/IPSOUT -> unconnected-(U2A-ELDOIN-Pad1)
- U2 pad 11: VCC_RTC -> unconnected-(U2A-N_VBUSEN-Pad11)
- U2 pad 12: PWR_ON -> unconnected-(U2A-PWRON-Pad12)
- U2 pad 13: /Power/IPSOUT -> Net-(U2B-VIN1)
- U2 pad 18: /Power/IPSOUT -> unconnected-(U2A-DLDOIN-Pad18)
- U2 pad 2: ELDO2 -> unconnected-(U2A-ELDO2-Pad2)
- U2 pad 23: /Power/IPSOUT -> Net-(U2C-VIN2)
- U2 pad 28: CPUX_FB -> VCC1V2_CPU
- U2 pad 29: AXP_IRQ -> unconnected-(U2A-IRQ-Pad29)
- U2 pad 3: ELDO3 -> unconnected-(U2A-ELDO3-Pad3)
- U2 pad 30: NTC -> unconnected-(U2A-TS-Pad30)
- U2 pad 31: Net-(U2A-GPIO1/PWREN) -> unconnected-(U2A-GPIO1/PWREN-Pad31)
- U2 pad 32: VCC3V3_AUDIO -> unconnected-(U2A-ALDO1-Pad32)
- U2 pad 33: /Power/IPSOUT -> unconnected-(U2A-ALDOIN-Pad33)
- U2 pad 37: Net-(U2A-GPIO0) -> unconnected-(U2A-GPIO0-Pad37)
- U2 pad 39: /Power/IPSOUT -> Net-(U2D-VIN3)
- U2 pad 43: AXP_PWROK -> unconnected-(U2A-PWROK-Pad43)
- U2 pad 44: AXP_SCL -> unconnected-(U2A-SCK-Pad44)
- U2 pad 45: AXP_SDA -> unconnected-(U2A-SDA-Pad45)
- U2 pad 46: VCC_RTC -> Net-(U2A-VCC_RTC)
- U2 pad 49: +BATT -> unconnected-(U2A-BATSENCE-Pad49)
- U2 pad 50: /Power/CHSENCEN -> unconnected-(U2A-LOADSENCE-Pad50)
- U2 pad 51: /Power/N_BATDRV -> unconnected-(U2A-N_BATDRV-Pad51)
- U2 pad 52: CHG_LED -> unconnected-(U2A-CHGLED-Pad52)
- U2 pad 53: /Power/IPSOUT -> unconnected-(U2A-PS-Pad53)
- U2 pad 54: /Power/IPSOUT -> unconnected-(U2A-PS-Pad54)
- U2 pad 57: /Power/CHSENCEP -> unconnected-(U2A-CHSENCEP-Pad57)
- U2 pad 58: /Power/CHSENCEN -> unconnected-(U2A-CHSENCEN-Pad58)
- U2 pad 59: GND -> unconnected-(U2A-PGND_CHG-Pad59)
- U2 pad 60: /Power/LX_CHG -> unconnected-(U2A-LX_CHG-Pad60)
- U2 pad 61: /Power/LX_CHG -> unconnected-(U2A-LX_CHG-Pad61)
- U2 pad 62: /Power/IPSOUT -> unconnected-(U2A-VIN_CHG-Pad62)
- U2 pad 63: /Power/IPSOUT -> unconnected-(U2A-VIN_CHG-Pad63)
- U2 pad 64: /Power/IPSOUT -> unconnected-(U2E-VIN4-Pad64)
- U2 pad 65: Net-(U2E-LX4) -> unconnected-(U2E-LX4-Pad65)
- U2 pad 66: GND -> unconnected-(U2E-PGND4-Pad66)
- U2 pad 67: DCDC4 -> unconnected-(U2E-DCDC4-Pad67)
- U2 pad 68: ELDO1 -> unconnected-(U2A-ELDO1-Pad68)
- U2 pad 9: /Power/IPSOUT -> Net-(U2F-VIN5)
- U9 pad 20: Net-(U9-INTB) -> unconnected-(U9-INTB-Pad20)
- U9 pad 21: /Ethernet/DVDD25 -> unconnected-(U9-DVDD33-Pad21)
- U9 pad 29: /Ethernet/PHYRSTB -> unconnected-(U9-PHYRSTB-Pad29)
- U9 pad 33: Net-(U9-PMEB) -> unconnected-(U9-PMEB-Pad33)
- U9 pad 37: VCC3V3 -> unconnected-(U9-DVDD33-Pad37)
- U9 pad 38: VCC3V3 -> unconnected-(U9-ENSWREG-Pad38)
- U9 pad 41: VCC3V3 -> unconnected-(U9-AVDD33-Pad41)
- U9 pad 42: /Ethernet/CKXTAL_OUT -> unconnected-(U9-CKXTAL1-Pad42)
- U9 pad 43: /Ethernet/CKXTAL_IN -> unconnected-(U9-CKXTAL2-Pad43)
- U9 pad 46: Net-(U9-CLK125) -> unconnected-(U9-CLK125-Pad46)
- U9 pad 6: VCC3V3 -> unconnected-(U9-AVDD33-Pad6)
