File: H3_SBC-backups/H3_SBC-2025-04-02_204858/Power.kicad_sch (KiCad schematic)
At the start: 82 parts, among them Q1 WPM1481-6/TR, U1 H3, U2 AXP223_C2997893

Commit message: small fixes
Parts:
- removed C14, C64, C72, C73, C76, C81: 10uF, symbol Device:C
- removed C65: 1nF, symbol Device:C
- removed C70, C71: 22uF, symbol Device:C
- removed C74, C77, C78, C82, C83: 1uF, symbol Device:C
- removed C75, C79, C80, C84, C85, C86: 0.1uF, symbol Device:C
- removed L7: 1.5uH, symbol Device:L
Connections:
- net GND: no longer U2.66 (PGND4)
- net IPSOUT: no longer C29.2, U2.64 (VIN4), U2.9 (VIN5)
- net DCDC4: no longer names the net of U2.67 (DCDC4)
- new net: C29.2, U2.9 (VIN5)
- no-connect marks 3 -> 7
Other:
- moved on the sheet: C1, C10, C13, C2, C27, C28, C29, C3, C30, C4, C5, C6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
