File: H3_SBC-backups/H3_SBC-2025-04-04_234245/Power.kicad_sch (KiCad schematic)
At the start: 82 parts, among them Q1 WPM1481-6/TR, U1 H3, U2 AXP223_C2997893

Commit message: small fixes
Parts:
- removed C73, C76, C81: 10uF, symbol Device:C
- removed C74, C77, C78, C82, C83: 1uF, symbol Device:C
- removed C75, C79, C80, C84, C85, C86: 0.1uF, symbol Device:C
Connections:
- net IPSOUT: no longer C29.2, U2.9 (VIN5)
- new net: C29.2, U2.9 (VIN5)
Other:
- moved on the sheet: C1, C10, C13, C2, C3, C4, C5, C6, C7, C8, C9, L1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
